Commit message: new urdf

File: bi_pedal_a1/urdf/robot.urdf.xacro (robot description, xacro)
@@ -4,4 +4,5 @@
     <xacro:arg name="HW_mode" default="mock"/> -->
     <xacro:include filename="robot_core.xacro"/>
+    <!-- <xacro:include filename="robot_core_2.xacro"/> -->
     <!-- <xacro:include filename="ros2_control.xacro"/> -->
     <!-- XACRO to handle multiple ros2_control hardware_interface plugins -->

File: bi_pedal_a1/urdf/robot_core.xacro (robot description, xacro)
@@ -27,5 +27,5 @@
             </geometry>
         </collision>
-        <inertial>
+        <!-- <inertial>
             <origin xyz="0 -0.00225 0.01017"/>
             <mass value="2.234" />
@@ -33,5 +33,5 @@
                     iyx="0.00000022295" iyy="0.05" iyz="0.000004933"
                     izx="0.0000001396" izy="0.000004933" izz="0.05" />
-        </inertial>
+        </inertial> -->
     </link>
     <joint name="base_joint" type="fixed">
@@ -57,5 +57,5 @@
             </geometry>
         </collision>
-        <inertial>
+        <!-- <inertial>
             <origin xyz="0.00262 0 0.04794"/>
             <mass value="0.3847" />
@@ -63,5 +63,5 @@
                     iyx="-0.0000013" iyy="0.0002" iyz="0.000000485"
                     izx="-0.000002522" izy="0.000000485" izz="0.0002" />
-        </inertial>
+        </inertial> -->
     </link>
     <joint name="left_hip_joint" type="revolute">
@@ -89,5 +89,5 @@
             </geometry>
         </collision>
-        <inertial>
+        <!-- <inertial>
             <origin xyz="-0.00262 0 0.04794"/>
             <mass value="0.3847" />
@@ -95,5 +95,5 @@
                     iyx="-0.0000013" iyy="0.0002" iyz="0.000000485"
                     izx="0.000003369" izy="-0.000000485" izz="0.0002" />
-        </inertial>
+        </inertial> -->
     </link>
     <joint name="right_hip_joint" type="revolute">
@@ -121,5 +121,5 @@
             </geometry>
         </collision>
-        <inertial>
+        <!-- <inertial>
             <origin xyz="0.0148 0 -0.201"/>
             <mass value="0.619" />
@@ -127,5 +127,5 @@
                     iyx="0.000001214" iyy="0.009" iyz="0.000009833"
                     izx="0.000031265" izy="0.000009833" izz="0.0002" />
-        </inertial>
+        </inertial> -->
     </link>
     <joint name="left_thigh_joint" type="revolute">
@@ -153,5 +153,5 @@
             </geometry>
         </collision>
-        <inertial>
+        <!-- <inertial>
             <origin xyz="-0.0139 0 -0.201"/>
             <mass value="0.619" />
@@ -159,5 +159,5 @@
                     iyx="0.000001214" iyy="0.009" iyz="0.000009833"
                     izx="0.000031265" izy="0.000009833" izz="0.0002" />
-        </inertial>
+        </inertial> -->
     </link>
     <joint name="right_thigh_joint" type="revolute">
@@ -185,5 +185,5 @@
             </geometry>
         </collision>
-        <inertial>
+        <!-- <inertial>
             <origin xyz="-0.0136 0 -0.2296"/>
             <mass value="0.542" />
@@ -191,5 +191,5 @@
                     iyx="0.000001214" iyy="0.005" iyz="0.000009833"
                     izx="0.000031265" izy="0.000009833" izz="0.002" />
-        </inertial>
+        </inertial> -->
     </link>
     <joint name="left_shin_joint" type="revolute">
@@ -217,5 +217,5 @@
             </geometry>
         </collision>
-        <inertial>
+        <!-- <inertial>
             <origin xyz="0.01466 0 -0.2296"/>
             <mass value="0.542" />
@@ -223,5 +223,5 @@
                     iyx="0.000001257" iyy="0.005" iyz="-0.000009833"
                     izx="-0.000007509" izy="-0.000009833" izz="0.002" />
-        </inertial>
+        </inertial> -->
     </link>
     <joint name="right_shin_joint" type="revolute">
@@ -249,5 +249,5 @@
             </geometry>
         </collision>
-        <inertial>
+        <!-- <inertial>
             <origin xyz="0.0049 0 -0.0351"/>
             <mass value="0.233" />
@@ -255,5 +255,5 @@
                     iyx="0.000000214" iyy="0.0002" iyz="0.000000194"
                     izx="-0.000045314" izy="0.000000194" izz="0.0001" />
-        </inertial>
+        </inertial> -->
     </link>
     <joint name="left_foot_joint" type="revolute">
@@ -281,5 +281,5 @@
             </geometry>
         </collision>
-        <inertial>
+        <!-- <inertial>
             <origin xyz="-0.00477 0 -0.0351"/>
             <mass value="0.233" />
@@ -287,5 +287,5 @@
                     iyx="-0.000000068" iyy="0.0002" iyz="-0.000000137"
                     izx="0.000045314" izy="-0.000000137" izz="0.0001" />
-        </inertial>
+        </inertial> -->
     </link>
     <joint name="right_foot_joint" type="revolute">

Commit message: updated urdf with independent inertial properties

File: bi_pedal_a1/urdf/robot.urdf.xacro (robot description, xacro)
@@ -3,6 +3,6 @@
     <!-- <xacro:arg name="cmd_mode" default="position"/>
     <xacro:arg name="HW_mode" default="mock"/> -->
-    <xacro:include filename="robot_core.xacro"/>
-    <!-- <xacro:include filename="robot_core_2.xacro"/> -->
+    <!-- <xacro:include filename="robot_core.xacro"/> -->
+    <xacro:include filename="robot_core_2.xacro"/>
     <!-- <xacro:include filename="ros2_control.xacro"/> -->
     <!-- XACRO to handle multiple ros2_control hardware_interface plugins -->

File: bi_pedal_a1/urdf/robot_core_2.xacro (robot description, xacro)
@@ -1,4 +1,5 @@
 <?xml version="1.0"?>
 <robot xmlns:xacro="http://www.ros.org/wiki/xacro">
+    <xacro:include filename="inertial_properties.xacro"/>
     <material name="grey">
         <color rgba="0.5 0.5 0.5 1"/>
@@ -27,11 +28,5 @@
             </geometry>
         </collision>
-        <!-- <inertial>
-            <origin xyz="0 -0.00225 0.01017"/>
-            <mass value="2.234" />
-            <inertia ixx="0.001" ixy="0.00000022295" ixz="0.0000001396"
-                    iyx="0.00000022295" iyy="0.05" iyz="0.000004933"
-                    izx="0.0000001396" izy="0.000004933" izz="0.05" />
-        </inertial> -->
+        <xacro:base_link_inertial/>
     </link>
     <joint name="base_joint" type="fixed">
@@ -57,11 +52,5 @@
             </geometry>
         </collision>
-        <!-- <inertial>
-            <origin xyz="0.00262 0 0.04794"/>
-            <mass value="0.3847" />
-            <inertia ixx="0.0004" ixy="-0.0000013" ixz="-0.000002522"
-                    iyx="-0.0000013" iyy="0.0002" iyz="0.000000485"
-                    izx="-0.000002522" izy="0.000000485" izz="0.0002" />
-        </inertial> -->
+        <xacro:left_hip_inertial/>
     </link>
     <joint name="left_hip_joint" type="revolute">
@@ -89,11 +78,5 @@
             </geometry>
         </collision>
-        <!-- <inertial>
-            <origin xyz="-0.00262 0 0.04794"/>
-            <mass value="0.3847" />
-            <inertia ixx="0.0004" ixy="-0.0000013" ixz="0.000003369"
-                    iyx="-0.0000013" iyy="0.0002" iyz="0.000000485"
-                    izx="0.000003369" izy="-0.000000485" izz="0.0002" />
-        </inertial> -->
+        <xacro:right_hip_inertial/>
     </link>
     <joint name="right_hip_joint" type="revolute">
@@ -121,11 +104,5 @@
             </geometry>
         </collision>
-        <!-- <inertial>
-            <origin xyz="0.0148 0 -0.201"/>
-            <mass value="0.619" />
-            <inertia ixx="0.009" ixy="0.000001214" ixz="0.000031265"
-                    iyx="0.000001214" iyy="0.009" iyz="0.000009833"
-                    izx="0.000031265" izy="0.000009833" izz="0.0002" />
-        </inertial> -->
+        <xacro:left_thigh_inertial/>
     </link>
     <joint name="left_thigh_joint" type="revolute">
@@ -153,11 +130,5 @@
             </geometry>
         </collision>
-        <!-- <inertial>
-            <origin xyz="-0.0139 0 -0.201"/>
-            <mass value="0.619" />
-            <inertia ixx="0.009" ixy="0.000001214" ixz="0.000031265"
-                    iyx="0.000001214" iyy="0.009" iyz="0.000009833"
-                    izx="0.000031265" izy="0.000009833" izz="0.0002" />
-        </inertial> -->
+        <xacro:right_thigh_inertial/>
     </link>
     <joint name="right_thigh_joint" type="revolute">
@@ -185,11 +156,5 @@
             </geometry>
         </collision>
-        <!-- <inertial>
-            <origin xyz="-0.0136 0 -0.2296"/>
-            <mass value="0.542" />
-            <inertia ixx="0.006" ixy="0.000001214" ixz="0.000031265"
-                    iyx="0.000001214" iyy="0.005" iyz="0.000009833"
-                    izx="0.000031265" izy="0.000009833" izz="0.002" />
-        </inertial> -->
+        <xacro:left_shin_inertial/>
     </link>
     <joint name="left_shin_joint" type="revolute">
@@ -217,11 +182,5 @@
             </geometry>
         </collision>
-        <!-- <inertial>
-            <origin xyz="0.01466 0 -0.2296"/>
-            <mass value="0.542" />
-            <inertia ixx="0.006" ixy="0.000001214" ixz="-0.000007509"
-                    iyx="0.000001257" iyy="0.005" iyz="-0.000009833"
-                    izx="-0.000007509" izy="-0.000009833" izz="0.002" />
-        </inertial> -->
+        <xacro:right_shin_inertial/>
     </link>
     <joint name="right_shin_joint" type="revolute">
@@ -249,11 +208,5 @@
             </geometry>
         </collision>
-        <!-- <inertial>
-            <origin xyz="0.0049 0 -0.0351"/>
-            <mass value="0.233" />
-            <inertia ixx="0.002" ixy="0.000000214" ixz="-0.000045314"
-                    iyx="0.000000214" iyy="0.0002" iyz="0.000000194"
-                    izx="-0.000045314" izy="0.000000194" izz="0.0001" />
-        </inertial> -->
+        <xacro:left_foot_inertial/>
     </link>
     <joint name="left_foot_joint" type="revolute">
@@ -281,11 +234,5 @@
             </geometry>
         </collision>
-        <!-- <inertial>
-            <origin xyz="-0.00477 0 -0.0351"/>
-            <mass value="0.233" />
-            <inertia ixx="0.002" ixy="-0.000000068" ixz="0.000045314"
-                    iyx="-0.000000068" iyy="0.0002" iyz="-0.000000137"
-                    izx="0.000045314" izy="-0.000000137" izz="0.0001" />
-        </inertial> -->
+        <xacro:right_foot_inertial/>
     </link>
     <joint name="right_foot_joint" type="revolute">
